File: HW2/ME 433 PCB/AndrewSaLoutos_pcb.brd (EAGLE design)
At the start: 50 x 50 mm, 23 parts

Commit message: Making progress on board layout
Parts:
- LED1: value (none) -> Green
- LED2: value (none) -> Red
- moved R4 65.0 mm to (42.0, 43.7), turned to 180 degrees
- moved LED2 55.6 mm to (32.1, 46.6)
- moved CRYSTAL_OSC 42.0 mm to (19.3, 19.9), turned to 270 degrees
- moved LED1 21.6 mm to (25.2, 46.7)
- moved U$8 20.2 mm to (47.5, 5.42)
- moved U$6 18.5 mm to (40.4, 3.49)
- moved R2 13.3 mm to (42.0, 47.9), turned to 180 degrees
- moved U$3 9.42 mm to (1.27, 47.0), turned to 270 degrees
- moved C3 5.33 mm to (19.4, 8.66)
- moved C1 2.61 mm to (36.2, 34.7)
- moved U$9 2.40 mm to (1.27, 34.3)
- moved U$10 1.50 mm to (48.8, 34.3)
- moved U$1 1.28 mm to (27.3, 22.5)
- moved C4 0.96 mm to (36.3, 15.2)
- moved C2 0.65 mm to (36.2, 23.5)

Commit message: Everything on the board, not very neat yet
Parts:
- moved C7 87.0 mm to (42.1, 32.2), turned to 90 degrees
- moved C6 57.2 mm to (34.6, 32.0), turned to 90 degrees
- moved C5 54.7 mm to (39.1, 18.5)
- moved U$7 49.8 mm to (36.8, 24.9), turned to 180 degrees
- moved R3 48.6 mm to (8.83, 34.9), turned to 270 degrees
- moved R1 38.5 mm to (5.37, 34.8), turned to 90 degrees
- moved U$8 14.7 mm to (33.0, 2.88), turned to 0 degrees
- moved CRYSTAL_OSC 12.1 mm to (8.17, 24.5)
- moved C3 11.0 mm to (8.79, 11.7)
- moved C1 10.8 mm to (25.6, 32.2)
- moved C2 10.2 mm to (26.0, 23.1)
- moved U$1 10.1 mm to (17.2, 22.7)
- moved C4 9.83 mm to (26.5, 14.9)
- moved RESET 9.30 mm to (15.1, 46.3)
- moved USER 8.83 mm to (6.11, 46.2)
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
Commit message: Ground plane
Parts:
- moved U$7 3.38 mm to (38.6, 22.1)
- moved C7 2.71 mm to (40.8, 29.8)
- moved C6 2.26 mm to (35.3, 29.9)
- moved C5 2.14 mm to (38.2, 16.5)
- moved LED2 1.41 mm to (32.4, 45.2)
- moved LED1 1.40 mm to (25.1, 45.3)
- moved CRYSTAL_OSC 1.32 mm to (9.45, 24.1)
- moved U$6 1.08 mm to (45.5, 8.79)
- moved C3 0.88 mm to (9.56, 11.2)
- moved U$8 0.62 mm to (33.6, 3.12)
Routing:
- added copper zone on layer 16, net GND

Commit message: Started traces
Parts:
- moved C4 9.44 mm to (27.0, 24.3), turned to 90 degrees
- moved C6 8.70 mm to (34.0, 38.5), turned to 180 degrees
- moved C7 8.66 mm to (42.1, 38.4), turned to 0 degrees
- moved C5 8.64 mm to (33.1, 9.55), turned to 180 degrees
- moved C2 7.52 mm to (33.5, 24.1)
- moved C1 6.62 mm to (26.4, 38.8)
- moved U$7 4.86 mm to (40.2, 26.6)
- moved C3 2.91 mm to (7.92, 8.84), turned to 90 degrees
- moved LED1 1.64 mm to (25.9, 46.8)
- moved LED2 1.50 mm to (32.2, 46.7), turned to 90 degrees
- moved U$1 0.12 mm to (17.2, 22.8)
Routing:
- net +3V3: track 0.00 -> 57.5 mm
- net +5V: track 0.00 -> 42.1 mm
- net B9: track 0.00 -> 33.0 mm
- net B8: track 0.00 -> 33.0 mm
- net B7: track 0.00 -> 33.0 mm
- net B15: track 0.00 -> 27.8 mm
- net B13: track 0.00 -> 27.8 mm
- net B14: track 0.00 -> 27.8 mm
- net N$6: track 0.00 -> 15.9 mm
- net N$17: track 0.00 -> 6.54 mm
- net N$11: track 0.00 -> 6.44 mm

Commit message: More traces
Parts:
- moved CRYSTAL_OSC 3.93 mm to (8.97, 20.2)
- moved U$8 1.05 mm to (33.6, 4.17)
- moved C5 0.30 mm to (33.1, 9.86)
Routing:
- net USBID: track 0.00 -> 38.5 mm
- net USBD-: track 0.00 -> 33.1 mm, vias 0 -> 2
- net USBD+: track 0.00 -> 24.7 mm, vias 0 -> 1
- net +3V3: track 57.5 -> 74.5 mm
- net B4/USER: track 0.00 -> 16.4 mm
- net A4/LED: track 0.00 -> 16.4 mm
- net N$11: track 6.44 -> 22.5 mm
- net N$1: track 0.00 -> 7.65 mm
- net N$2: track 0.00 -> 5.05 mm
- net N$3: track 0.00 -> 4.89 mm
- net +5V: track 42.1 -> 40.9 mm
Changed lines of the file:
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@@
 </element>
 <element name="C4" library="433_lib" package="E2,5-6" value="10uF" x="27.005" y="24.32" rot="R90"/>
-<element name="C5" library="433_lib" package="C050-030X075" value="0.1uF" x="33.085" y="9.555" rot="R180"/>
+<element name="C5" library="433_lib" package="C050-030X075" value="0.1uF" x="33.06" y="9.855" rot="R180"/>
 <element name="C6" library="433_lib" package="C050-030X075" value="0.1uF" x="34.025" y="38.455" rot="R180"/>
 <element name="C7" library="433_lib" package="E2,5-6" value="10uF" x="42.135" y="38.395"/>
@@
 <element name="R4" library="433_lib" package="0207/10" value="330" x="42.025" y="43.67" rot="R180"/>
 <element name="U$1" library="433_lib" package="DIL28-3" value="PIC32MX250F128B" x="17.225" y="22.8" rot="R270"/>
-<element name="CRYSTAL_OSC" library="433_lib" package="1X03" value="8 MHz" x="9.445" y="24.14" rot="R270"/>
+<element name="CRYSTAL_OSC" library="433_lib" package="1X03" value="8 MHz" x="8.97" y="20.24" rot="R270"/>
 <element name="U$3" library="433_lib" package="1X05" value="PICKIT_CONN" x="1.27" y="46.99" rot="R270"/>
 <element name="RESET" library="433_lib" package="PUSH_BUTTON" value="PUSH_BUTTON" x="15.115" y="46.265"/>
@@
 </element>
 <element name="U$7" library="433_lib" package="TO92" value="" x="40.24" y="26.625" rot="R180"/>
-<element name="U$8" library="433_lib" package="SLIDE" value="SLIDE" x="33.625" y="3.115" smashed="yes">
-<attribute name="NAME" x="28.98" y="5.655" size="1.27" layer="21"/>
-<attribute name="VALUE" x="33.38" y="5.715" size="1.27" layer="21"/>
+<element name="U$8" library="433_lib" package="SLIDE" value="SLIDE" x="33.6" y="4.165" smashed="yes">
+<attribute name="NAME" x="28.955" y="6.705" size="1.27" layer="21"/>
+<attribute name="VALUE" x="33.355" y="6.765" size="1.27" layer="21"/>
 </element>
 <element name="U$9" library="433_lib" package="8PIN_HEADER" value="8PIN_HEADER" x="1.27" y="34.29" rot="R270"/>
@@
 <contactref element="U$6" pad="VBUS"/>
 <contactref element="U$8" pad="2"/>
-<wire x1="33.625" y1="3.115" x2="33.625" y2="4.875" width="0.254" layer="16"/>
-<wire x1="33.625" y1="4.875" x2="38.065" y2="4.875" width="0.254" layer="16"/>
-<wire x1="38.065" y1="4.875" x2="40.385" y2="7.195" width="0.254" layer="16"/>
+<wire x1="33.6" y1="4.165" x2="33.625" y2="5.7" width="0.254" layer="16"/>
+<wire x1="33.625" y1="5.7" x2="38.14" y2="5.7" width="0.254" layer="16"/>
+<wire x1="38.14" y1="5.7" x2="40.385" y2="7.195" width="0.254" layer="16"/>
 <wire x1="40.385" y1="7.195" x2="40.385" y2="7.19" width="0.254" layer="16"/>
 <wire x1="40.385" y1="7.19" x2="41.7" y2="5.875" width="0.254" layer="16"/>
@@
 <wire x1="47.498" y1="15.98394375" x2="47.498" y2="17.78" width="0.254" layer="16"/>
 <wire x1="47.498" y1="17.78" x2="48.768" y2="19.05" width="0.254" layer="16"/>
-<wire x1="33.625" y1="4.875" x2="22.45" y2="4.875" width="0.254" layer="16"/>
-<wire x1="22.45" y1="4.875" x2="21.035" y2="6.29" width="0.254" layer="16"/>
+<wire x1="33.625" y1="5.7" x2="22.45" y2="5.7" width="0.254" layer="16"/>
+<wire x1="22.45" y1="5.7" x2="21.035" y2="6.29" width="0.254" layer="16"/>
 </signal>
 <signal name="GND">
@@
 <wire x1="26.41" y1="41.3" x2="23.025" y2="41.3" width="0.254" layer="16"/>
 <wire x1="23.025" y1="41.3" x2="21.035" y2="39.31" width="0.254" layer="16"/>
+<wire x1="13.415" y1="8.83" x2="10.465" y2="8.83" width="0.254" layer="1"/>
+<wire x1="10.465" y1="8.83" x2="7.915" y2="11.38" width="0.254" layer="1"/>
+<wire x1="7.915" y1="11.38" x2="7.915" y2="12.405" width="0.254" layer="1"/>
+<wire x1="7.915" y1="12.405" x2="1.27" y2="19.05" width="0.254" layer="1"/>
 <wire x1="8.83" y1="29.795" x2="21.035" y2="26.61" width="0" layer="19" extent="1-1"/>
 <wire x1="1.27" y1="19.05" x2="8.83" y2="29.795" width="0" layer="19" extent="1-1"/>
-<wire x1="7.915" y1="11.38" x2="1.27" y2="19.05" width="0" layer="19" extent="1-1"/>
-<wire x1="13.415" y1="8.83" x2="7.915" y2="11.38" width="0" layer="19" extent="1-1"/>
 <wire x1="1.27" y1="44.45" x2="8.83" y2="29.795" width="0" layer="19" extent="1-1"/>
 </signal>
@@
 <contactref element="U$1" pad="20"/>
 <contactref element="C4" pad="+"/>
-<wire x1="21.035" y1="18.99" x2="27.005" y2="23.05" width="0" layer="19" extent="1-1"/>
+<wire x1="21.035" y1="18.99" x2="22.945" y2="18.99" width="0.254" layer="1"/>
+<wire x1="22.945" y1="18.99" x2="27.005" y2="23.05" width="0.254" layer="1"/>
 </signal>
 <signal name="N$2">
 <contactref element="CRYSTAL_OSC" pad="1"/>
 <contactref element="U$1" pad="9"/>
-<wire x1="13.415" y1="18.99" x2="9.445" y2="24.14" width="0" layer="19" extent="1-1"/>
+<wire x1="13.415" y1="18.99" x2="9.97" y2="18.99" width="0.254" layer="1"/>
+<wire x1="9.97" y1="18.99" x2="8.97" y2="20.24" width="0.254" layer="1"/>
 </signal>
 <signal name="N$3">
 <contactref element="CRYSTAL_OSC" pad="3"/>
 <contactref element="U$1" pad="10"/>
-<wire x1="9.445" y1="19.06" x2="13.415" y2="16.45" width="0" layer="19" extent="1-1"/>
+<wire x1="13.415" y1="16.45" x2="10.61" y2="16.45" width="0.254" layer="16"/>
+<wire x1="10.61" y1="16.45" x2="8.97" y2="15.16" width="0.254" layer="16"/>
 </signal>
 <signal name="N$6">
@@
 <contactref element="C5" pad="1"/>
 <contactref element="U$8" pad="3"/>
-<wire x1="35.625" y1="9.555" x2="35.625" y2="3.115" width="0.254" layer="1"/>
-<wire x1="35.625" y1="9.555" x2="40.24" y2="24.72" width="0" layer="19" extent="1-1"/>
+<wire x1="35.6" y1="9.855" x2="35.6" y2="4.165" width="0.254" layer="1"/>
+<wire x1="35.6" y1="9.855" x2="35.6" y2="20.08" width="0.254" layer="16"/>
+<wire x1="35.6" y1="20.08" x2="40.24" y2="24.72" width="0.254" layer="16"/>
 </signal>
 <signal name="N$17">
@@
 <contactref element="U$1" pad="14"/>
 <contactref element="U$6" pad="ID"/>
-<wire x1="13.415" y1="6.29" x2="41.585" y2="9.595" width="0" layer="19" extent="1-1"/>
+<wire x1="13.415" y1="6.29" x2="13.415" y2="4.365" width="0.254" layer="1"/>
+<wire x1="13.415" y1="4.365" x2="15.24" y2="2.54" width="0.254" layer="1"/>
+<wire x1="40.69" y1="2.54" x2="42.9" y2="4.75" width="0.254" layer="1"/>
+<wire x1="42.9" y1="4.75" x2="42.9" y2="8.28" width="0.254" layer="1"/>
+<wire x1="42.9" y1="8.28" x2="41.585" y2="9.595" width="0.254" layer="1"/>
+<wire x1="15.24" y1="2.54" x2="40.69" y2="2.54" width="0.254" layer="1"/>
 </signal>
 <signal name="USBD+">
 <contactref element="U$1" pad="21"/>
 <contactref element="U$6" pad="D+"/>
-<wire x1="21.035" y1="21.53" x2="40.385" y2="8.795" width="0" layer="19" extent="1-1"/>
+<wire x1="40.385" y1="8.795" x2="38.405" y2="8.795" width="0.254" layer="1"/>
+<wire x1="38.405" y1="8.795" x2="33.775" y2="13.425" width="0.254" layer="1"/>
+<wire x1="33.75" y1="13.45" x2="33.775" y2="13.425" width="0.254" layer="1"/>
+<wire x1="33.775" y1="13.425" x2="33.75" y2="13.45" width="0.254" layer="1"/>
+<via x="33.775" y="13.425" extent="1-16" drill="0.6"/>
+<wire x1="33.775" y1="13.425" x2="29.14" y2="13.425" width="0.254" layer="16"/>
+<wire x1="29.14" y1="13.425" x2="21.035" y2="21.53" width="0.254" layer="16"/>
 </signal>
 <signal name="USBD-">
 <contactref element="U$1" pad="22"/>
 <contactref element="U$6" pad="D-"/>
-<wire x1="21.035" y1="24.07" x2="41.585" y2="7.995" width="0" layer="19" extent="1-1"/>
+<wire x1="41.585" y1="7.995" x2="43.42" y2="7.995" width="0.254" layer="16"/>
+<wire x1="43.42" y1="7.995" x2="44.125" y2="8.7" width="0.254" layer="16"/>
+<wire x1="44.125" y1="8.7" x2="44.125" y2="9.9" width="0.254" layer="16"/>
+<wire x1="44.125" y1="9.9" x2="37.575" y2="16.45" width="0.254" layer="16"/>
+<wire x1="37.55" y1="16.475" x2="37.575" y2="16.45" width="0.254" layer="16"/>
+<wire x1="37.575" y1="16.45" x2="37.55" y2="16.475" width="0.254" layer="16"/>
+<via x="37.575" y="16.45" extent="1-16" drill="0.6"/>
+<wire x1="37.575" y1="16.45" x2="33.775" y2="16.45" width="0.254" layer="1"/>
+<wire x1="33.75" y1="16.45" x2="33.775" y2="16.45" width="0.254" layer="1"/>
+<wire x1="33.775" y1="16.45" x2="33.75" y2="16.45" width="0.254" layer="1"/>
+<via x="33.775" y="16.45" extent="1-16" drill="0.6"/>
+<wire x1="33.775" y1="16.45" x2="28.655" y2="16.45" width="0.254" layer="16"/>
+<wire x1="28.655" y1="16.45" x2="21.035" y2="24.07" width="0.254" layer="16"/>
 </signal>
 <signal name="A4/LED">
@@
 <contactref element="U$1" pad="12"/>
 <contactref element="LED1" pad="A"/>
+<wire x1="13.415" y1="11.37" x2="11.49" y2="11.37" width="0.254" layer="1"/>
+<wire x1="11.49" y1="11.37" x2="1.27" y2="21.59" width="0.254" layer="1"/>
 <wire x1="1.27" y1="21.59" x2="24.585" y2="46.795" width="0" layer="19" extent="1-1"/>
-<wire x1="13.415" y1="11.37" x2="1.27" y2="21.59" width="0" layer="19" extent="1-1"/>
 </signal>
 <signal name="B4/USER">
@@
 <contactref element="USER" pad="3"/>
 <contactref element="U$1" pad="11"/>
+<wire x1="13.415" y1="13.91" x2="11.49" y2="13.91" width="0.254" layer="1"/>
+<wire x1="11.49" y1="13.91" x2="1.27" y2="24.13" width="0.254" layer="1"/>
 <wire x1="1.27" y1="24.13" x2="11.185" y2="46.245" width="0" layer="19" extent="1-1"/>
-<wire x1="13.415" y1="13.91" x2="1.27" y2="24.13" width="0" layer="19" extent="1-1"/>
 </signal>
 <signal name="B3">

Commit message: Traces finished
Routing:
- net +3V3: track 74.5 -> 148.0 mm
- net A4/LED: track 16.4 -> 58.8 mm
- net B4/USER: track 16.4 -> 52.1 mm
- net N$9: track 0.00 -> 33.7 mm
- net N$7: track 0.00 -> 15.3 mm
- net N$8: track 0.00 -> 15.3 mm
- net B3: track 0.00 -> 14.2 mm
- net B2: track 0.00 -> 14.2 mm
- net A0: track 0.00 -> 13.2 mm
- net A1: track 0.00 -> 13.2 mm
- net N$4: track 0.00 -> 6.67 mm
Changed lines of the file:
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@@
 <wire x1="26.24" y1="27.94" x2="24.825" y2="26.6" width="0.254" layer="1"/>
 <wire x1="24.825" y1="26.6" x2="21.475" y2="26.6" width="0.254" layer="1"/>
-<wire x1="21.475" y1="26.6" x2="21.035" y2="26.61" width="0.254" layer="1"/>
+<wire x1="21.035" y1="26.61" x2="21.475" y2="26.6" width="0.254" layer="1"/>
 <wire x1="38.97" y1="26.625" x2="38.97" y2="36.5" width="0.254" layer="16"/>
 <wire x1="39.335" y1="36.865" x2="38.97" y2="36.5" width="0.254" layer="16"/>
@@
 <wire x1="26.41" y1="41.3" x2="23.025" y2="41.3" width="0.254" layer="16"/>
 <wire x1="23.025" y1="41.3" x2="21.035" y2="39.31" width="0.254" layer="16"/>
-<wire x1="13.415" y1="8.83" x2="10.465" y2="8.83" width="0.254" layer="1"/>
+<wire x1="10.465" y1="8.83" x2="13.415" y2="8.83" width="0.254" layer="1"/>
 <wire x1="10.465" y1="8.83" x2="7.915" y2="11.38" width="0.254" layer="1"/>
 <wire x1="7.915" y1="11.38" x2="7.915" y2="12.405" width="0.254" layer="1"/>
 <wire x1="7.915" y1="12.405" x2="1.27" y2="19.05" width="0.254" layer="1"/>
-<wire x1="8.83" y1="29.795" x2="21.035" y2="26.61" width="0" layer="19" extent="1-1"/>
-<wire x1="1.27" y1="19.05" x2="8.83" y2="29.795" width="0" layer="19" extent="1-1"/>
-<wire x1="1.27" y1="44.45" x2="8.83" y2="29.795" width="0" layer="19" extent="1-1"/>
+<wire x1="13.415" y1="8.83" x2="17.45" y2="8.83" width="0.254" layer="1"/>
+<wire x1="17.45" y1="8.83" x2="18.855" y2="10.435" width="0.254" layer="1"/>
+<wire x1="18.855" y1="10.435" x2="18.88" y2="24.88" width="0.254" layer="1"/>
+<wire x1="18.88" y1="24.88" x2="21.035" y2="26.61" width="0.254" layer="1"/>
+<wire x1="1.27" y1="19.05" x2="3.81" y2="19.05" width="0.254" layer="16"/>
+<wire x1="3.81" y1="19.05" x2="10.16" y2="25.4" width="0.254" layer="16"/>
+<wire x1="10.16" y1="25.4" x2="10.16" y2="28.465" width="0.254" layer="16"/>
+<wire x1="8.83" y1="29.795" x2="10.16" y2="28.465" width="0.254" layer="16"/>
+<wire x1="1.27" y1="44.45" x2="5.08" y2="48.26" width="0.254" layer="16"/>
+<wire x1="5.08" y1="48.26" x2="29.375" y2="48.26" width="0.254" layer="16"/>
+<wire x1="29.375" y1="48.26" x2="32.195" y2="45.44" width="0.254" layer="16"/>
 </signal>
 <signal name="N$1">
@@
 <contactref element="U$3" pad="5"/>
 <contactref element="U$1" pad="5"/>
-<wire x1="1.27" y1="36.83" x2="13.415" y2="29.15" width="0" layer="19" extent="1-1"/>
+<wire x1="1.27" y1="36.83" x2="5.08" y2="33.02" width="0.254" layer="16"/>
+<wire x1="5.08" y1="33.02" x2="9.545" y2="33.02" width="0.254" layer="16"/>
+<wire x1="9.545" y1="33.02" x2="13.415" y2="29.15" width="0.254" layer="16"/>
 </signal>
 <signal name="N$8">
 <contactref element="U$3" pad="4"/>
 <contactref element="U$1" pad="4"/>
-<wire x1="1.27" y1="39.37" x2="13.415" y2="31.69" width="0" layer="19" extent="1-1"/>
+<wire x1="1.27" y1="39.37" x2="5.08" y2="35.56" width="0.254" layer="16"/>
+<wire x1="5.08" y1="35.56" x2="9.545" y2="35.56" width="0.254" layer="16"/>
+<wire x1="9.545" y1="35.56" x2="13.415" y2="31.69" width="0.254" layer="16"/>
 </signal>
 <signal name="N$9">
@@
 <contactref element="R3" pad="1"/>
 <contactref element="RESET" pad="3"/>
-<wire x1="13.415" y1="39.31" x2="20.195" y2="46.265" width="0" layer="19" extent="1-1"/>
-<wire x1="8.83" y1="39.955" x2="13.415" y2="39.31" width="0" layer="19" extent="1-1"/>
-<wire x1="1.27" y1="46.99" x2="8.83" y2="39.955" width="0" layer="19" extent="1-1"/>
+<wire x1="8.83" y1="39.955" x2="10.695" y2="39.305" width="0.254" layer="1"/>
+<wire x1="10.695" y1="39.305" x2="13.415" y2="39.31" width="0.254" layer="1"/>
+<wire x1="13.415" y1="47.285" x2="13.415" y2="39.31" width="0.254" layer="1"/>
+<wire x1="13.415" y1="47.285" x2="14.69" y2="48.26" width="0.254" layer="1"/>
+<wire x1="18.225" y1="48.26" x2="20.195" y2="46.265" width="0.254" layer="1"/>
+<wire x1="14.69" y1="48.26" x2="18.225" y2="48.26" width="0.254" layer="1"/>
+<wire x1="1.27" y1="46.99" x2="3.81" y2="46.99" width="0.254" layer="1"/>
+<wire x1="3.81" y1="46.99" x2="5.08" y2="48.26" width="0.254" layer="1"/>
+<wire x1="5.08" y1="48.26" x2="12.44" y2="48.26" width="0.254" layer="1"/>
+<wire x1="12.44" y1="48.26" x2="13.415" y2="47.285" width="0.254" layer="1"/>
 </signal>
 <signal name="N$4">
 <contactref element="R1" pad="2"/>
 <contactref element="USER" pad="1"/>
-<wire x1="5.37" y1="39.875" x2="6.105" y2="46.245" width="0" layer="19" extent="1-1"/>
+<wire x1="6.105" y1="46.245" x2="6.105" y2="40.61" width="0.254" layer="1"/>
+<wire x1="6.105" y1="40.61" x2="5.37" y2="39.875" width="0.254" layer="1"/>
 </signal>
 <signal name="N$11">
@@
 <wire x1="13.415" y1="11.37" x2="11.49" y2="11.37" width="0.254" layer="1"/>
 <wire x1="11.49" y1="11.37" x2="1.27" y2="21.59" width="0.254" layer="1"/>
-<wire x1="1.27" y1="21.59" x2="24.585" y2="46.795" width="0" layer="19" extent="1-1"/>
+<wire x1="24.585" y1="46.795" x2="23.935" y2="46.795" width="0.254" layer="1"/>
+<wire x1="23.935" y1="46.795" x2="17.78" y2="40.64" width="0.254" layer="1"/>
+<wire x1="17.78" y1="12.405" x2="16.75" y2="11.375" width="0.254" layer="1"/>
+<wire x1="16.75" y1="11.375" x2="13.42" y2="11.375" width="0.254" layer="1"/>
+<wire x1="13.42" y1="11.375" x2="13.415" y2="11.37" width="0.254" layer="1"/>
+<wire x1="17.78" y1="40.64" x2="17.78" y2="12.405" width="0.254" layer="1"/>
 </signal>
 <signal name="B4/USER">
@@
 <wire x1="13.415" y1="13.91" x2="11.49" y2="13.91" width="0.254" layer="1"/>
 <wire x1="11.49" y1="13.91" x2="1.27" y2="24.13" width="0.254" layer="1"/>
-<wire x1="1.27" y1="24.13" x2="11.185" y2="46.245" width="0" layer="19" extent="1-1"/>
+<wire x1="13.415" y1="13.91" x2="13.43" y2="13.925" width="0.254" layer="16"/>
+<wire x1="11.185" y1="46.245" x2="11.185" y2="45.915" width="0.254" layer="16"/>
+<wire x1="11.185" y1="45.915" x2="16.4" y2="40.7" width="0.254" layer="16"/>
+<wire x1="16.4" y1="40.7" x2="16.4" y2="16.895" width="0.254" layer="16"/>
+<wire x1="16.4" y1="16.895" x2="13.415" y2="13.91" width="0.254" layer="16"/>
 </signal>
 <signal name="B3">
 <contactref element="U$9" pad="4"/>
 <contactref element="U$1" pad="7"/>
-<wire x1="1.27" y1="26.67" x2="13.415" y2="24.07" width="0" layer="19" extent="1-1"/>
+<wire x1="1.27" y1="26.67" x2="5.08" y2="22.86" width="0.254" layer="1"/>
+<wire x1="5.08" y1="22.86" x2="12.205" y2="22.86" width="0.254" layer="1"/>
+<wire x1="12.205" y1="22.86" x2="13.415" y2="24.07" width="0.254" layer="1"/>
 </signal>
 <signal name="B2">
 <contactref element="U$9" pad="3"/>
 <contactref element="U$1" pad="6"/>
-<wire x1="1.27" y1="29.21" x2="13.415" y2="26.61" width="0" layer="19" extent="1-1"/>
+<wire x1="1.27" y1="29.21" x2="5.08" y2="25.4" width="0.254" layer="1"/>
+<wire x1="5.08" y1="25.4" x2="12.205" y2="25.4" width="0.254" layer="1"/>
+<wire x1="12.205" y1="25.4" x2="13.415" y2="26.61" width="0.254" layer="1"/>
 </signal>
 <signal name="A1">
 <contactref element="U$9" pad="2"/>
 <contactref element="U$1" pad="3"/>
-<wire x1="1.27" y1="31.75" x2="13.415" y2="34.23" width="0" layer="19" extent="1-1"/>
+<wire x1="1.27" y1="31.75" x2="10.935" y2="31.75" width="0.254" layer="1"/>
+<wire x1="10.935" y1="31.75" x2="13.415" y2="34.23" width="0.254" layer="1"/>
 </signal>
 <signal name="A0">
 <contactref element="U$9" pad="1"/>
 <contactref element="U$1" pad="2"/>
-<wire x1="1.27" y1="34.29" x2="13.415" y2="36.77" width="0" layer="19" extent="1-1"/>
+<wire x1="1.27" y1="34.29" x2="10.935" y2="34.29" width="0.254" layer="1"/>
+<wire x1="10.935" y1="34.29" x2="13.415" y2="36.77" width="0.254" layer="1"/>
 </signal>
 <signal name="B7">
